Commit message: fork.urdf.xacro: changed the origin of the inertia

File: rbares_description/urdf/elevator/fork.urdf.xacro (robot description, xacro)
@@ -16,5 +16,5 @@
      <link name="${prefix}fork_link">
        <inertial>
-         <origin xyz="-0.581270 0.00000 0.012941" />
+         <origin xyz="-0.381270 0.00000 0.012941" />
          <mass value="${fork_mass}" />
          <solid_cuboid_inertia m="${fork_mass}" h="${fork_width}" d="${fork_height}" w="${fork_length}"/>
