Commit message: projection.urdf.xacro: changed mass

File: rbares_description/urdf/bases/protection.urdf.xacro (robot description, xacro)
@@ -15,5 +15,5 @@
      </collision>
      <inertial>
-       <mass value="0.001" />
+       <mass value="0.01" />
        <origin xyz="0 0 0"/>
        <solid_cuboid_inertia m="0.001" h="0.001" d="0.001" w="0.001"/>
