Commit message: can run on real robot

File: rbares_description/urdf/bases/battery_case.urdf.xacro (robot description, xacro)
@@ -20,5 +20,6 @@
   </xacro:macro>
  <xacro:macro name="battery_case" params="prefix parent *origin">
-  <joint name="${prefix}elevator_joint" type="prismatic">
+  <!-- joint name="${prefix}elevator_joint" type="prismatic"-->
+  <joint name="${prefix}elevator_joint" type="fixed">
     <xacro:insert_block name="origin" />
     <parent link="${parent}"/>

File: rbares_description/urdf/elevator/fork.urdf.xacro (robot description, xacro)
@@ -8,5 +8,6 @@
 	<xacro:property name="fork_mass" value="1" />
   <xacro:macro name="fork" params="prefix parent *origin">
-    <joint name="${prefix}fork_joint" type="prismatic">
+    <!-- joint name="${prefix}fork_joint" type="prismatic"-->
+    <joint name="${prefix}fork_joint" type="fixed">
        <xacro:insert_block name="origin" />
        <parent link="${parent}"/>

Commit message: rbares_description: removed error and warning msgs

File: rbares_description/urdf/bases/battery_case.urdf.xacro (robot description, xacro)
@@ -20,6 +20,5 @@
   </xacro:macro>
  <xacro:macro name="battery_case" params="prefix parent *origin">
-  <!-- joint name="${prefix}elevator_joint" type="prismatic"-->
-  <joint name="${prefix}elevator_joint" type="fixed">
+  <joint name="${prefix}elevator_joint" type="prismatic">
     <xacro:insert_block name="origin" />
     <parent link="${parent}"/>

File: rbares_description/urdf/bases/rbares.urdf.xacro (robot description, xacro)
@@ -7,8 +7,8 @@
   <!-- BASE FOOTPRINT -->
   <link name="${prefix}base_footprint">
-    <inertial>
+    <!--inertial>
       <mass value="0.0001"/>
       <inertia ixx="0.0001" ixy="0" ixz="0" iyy="0.0001" iyz="0" izz="0.0001"/>
-    </inertial>
+    </inertial-->
   </link>
   <joint name="${prefix}base_footprint_joint" type="fixed">

File: rbares_description/urdf/elevator/fork.urdf.xacro (robot description, xacro)
@@ -43,5 +43,5 @@
        </collision>
      </link>
-     <transmission name="${prefix}fork_transmission">
+     <!--transmission name="${prefix}fork_transmission">
        <type>transmission_interface/SimpleTransmission</type>
        <joint name="${prefix}fork_joint">
@@ -52,5 +52,5 @@
          <mechanicalReduction>${traction_mechanical_reduction}</mechanicalReduction>
        </actuator>
-     </transmission>
+     </transmission-->
      <!-- ***************** -->
      <!-- GAZEBO PROPERTIES -->

Commit message: updated config with the version of the robot

File: rbares_description/urdf/bases/battery_case.urdf.xacro (robot description, xacro)
@@ -20,6 +20,6 @@
   </xacro:macro>
  <xacro:macro name="battery_case" params="prefix parent *origin">
-  <!-- joint name="${prefix}elevator_joint" type="prismatic"-->
-  <joint name="${prefix}elevator_joint" type="fixed">
+  <joint name="${prefix}elevator_joint" type="prismatic">
+  <!--joint name="${prefix}elevator_joint" type="fixed"-->
     <xacro:insert_block name="origin" />
     <parent link="${parent}"/>
