Commit message: rbares_description: removed footprint inertia

File: rbares_description/urdf/bases/rbares.urdf.xacro (robot description, xacro)
@@ -6,10 +6,5 @@
   <xacro:macro name="rbares" params="prefix publish_bf">
   <!-- BASE FOOTPRINT -->
-  <link name="${prefix}base_footprint">
-    <inertial>
-      <mass value="0.0001"/>
-      <inertia ixx="0.0001" ixy="0" ixz="0" iyy="0.0001" iyz="0" izz="0.0001"/>
-    </inertial>
-  </link>
+  <link name="${prefix}base_footprint"/>
   <joint name="${prefix}base_footprint_joint" type="fixed">
     <origin xyz="${base_link_origin}" rpy="0 0 0" />
