Commit message: rbares_description: minor changes

File: rbares_description/urdf/bases/front_case.urdf.xacro (robot description, xacro)
@@ -48,6 +48,5 @@
 				<origin xyz="0.1993 0.43 0.197" rpy="0 0 0" />
 		 </xacro:line_projector-->
-		 <xacro:led prefix="${prefix}">
-		 </xacro:led>
+		 <xacro:led prefix="${prefix}"/>
     <gazebo reference="${prefix}front_case_link">
       <visual>

File: rbares_description/urdf/led/led2.urdf.xacro (robot description, xacro)
@@ -52,9 +52,9 @@
           </material>
         </visual>
-        <light name="${prefix}led_light" type="point">
+        <!--light name="${prefix}led_light" type="point">
           <pose>0 0 0 0 0 0</pose>
           <attenuation>
             <range>20</range>
-            <!--linear>0.10</linear-->
+            <!- -linear>0.10</linear- ->
           </attenuation>
           <diffuse>0 0 0 1</diffuse>
@@ -77,5 +77,5 @@
             <izz>0.0001</izz>
           </inertia>
-        </inertial>
+        </inertial-->
       </link>
       <!--plugin name='light_control' filename='libLedPlugin.so'>
