Commit message: rbares_description: realistic steer joint velocity

File: rbares_description/urdf/wheels/motor_wheel.urdf.xacro (robot description, xacro)
@@ -9,5 +9,5 @@
   <xacro:property name="steer_joint_friction" value="1000.0" />
   <xacro:property name="steer_joint_effort_limit" value="9999.0" />
-  <xacro:property name="steer_joint_velocity_limit" value="20" />
+  <xacro:property name="steer_joint_velocity_limit" value="1" />
   <xacro:property name="steer_mechanical_reduction" value="1.0" />
   <xacro:property name="steer_joint_position_limit" value="1.56" />
