Commit message: led2.urdf.xacro: changed inertia values

File: rbares_description/urdf/led/led2.urdf.xacro (robot description, xacro)
@@ -38,4 +38,16 @@
           </spot>
         </light>
+        <inertial>
+          <pose>0 0 0 0 0 0</pose>
+          <mass>0.1</mass>
+          <inertia>
+            <ixx>0.0001</ixx>
+            <ixy>-0</ixy>
+            <ixz>0</ixz>
+            <iyy>0.0001</iyy>
+            <iyz>0</iyz>
+            <izz>0.0001</izz>
+          </inertia>
+  </inertial>
       </link>
       <!--plugin name='light_control' filename='libLedPlugin.so'>

Commit message: rbares_description: added the three led stripes and the gazebo plugin

File: rbares_description/urdf/led/led2.urdf.xacro (robot description, xacro)
@@ -8,11 +8,39 @@
     </joint>
     <model name="light_model">
-      <pose>1.5207 0 0.68 0 0 0</pose>
+      <pose>0 0 0 0 0 0</pose>
       <link name="${prefix}light_link">
-        <visual name="${prefix}led_light">
-          <pose>0 0 0 0 0 0</pose>
+        <visual name="robot_visual">
+          <pose>1.77 0 0.71 0 0 0</pose>
           <geometry>
             <box>
-              <size>0.35 0.568 0.01</size>
+              <size>0.01 0.4 0.01</size>
+            </box>
+          </geometry>
+          <material>
+            <ambient>1 1 1 1</ambient>
+            <diffuse>1 1 1 1</diffuse>
+            <specular>1 1 1 1</specular>
+            <emissive>0 0 0 1</emissive>
+          </material>
+        </visual>
+        <visual name="robot_visual_2">
+          <pose>1.49 0.285 0.71 0 0 0</pose>
+          <geometry>
+            <box>
+              <size>0.4 0.01 0.01</size>
+            </box>
+          </geometry>
+          <material>
+            <ambient>1 1 1 1</ambient>
+            <diffuse>1 1 1 1</diffuse>
+            <specular>1 1 1 1</specular>
+            <emissive>0 0 0 1</emissive>
+          </material>
+        </visual>
+        <visual name="robot_visual_3">
+          <pose>1.49 -0.285 0.71 0 0 0</pose>
+          <geometry>
+            <box>
+              <size>0.4 0.01 0.01</size>
             </box>
           </geometry>
@@ -49,13 +77,12 @@
             <izz>0.0001</izz>
           </inertia>
-  </inertial>
+        </inertial>
       </link>
       <!--plugin name='light_control' filename='libLedPlugin.so'>
-       <enable>true</enable>
         <light>
-          <id>light_link/light_source</id>
+          <id>robot_light_link/robot_led_light</id>
             <enable>true</enable>
             <duration>1</duration>
-            <interval>0.5</interval>
+            <interval>1</interval>
             <color>1 0 0</color>
             <attenuation>
@@ -65,4 +92,16 @@
         </light>
       </plugin-->
+      <plugin name='robotnik_gazebo_set_visual' filename='librobotnik_gazebo_set_visual.so'>
+        <modelName>robot_light_link</modelName>
+        <visual>
+          <visualName>robot_visual</visualName>
+        </visual>
+        <visual>
+          <visualName>robot_visual_2</visualName>
+        </visual>
+        <visual>
+          <visualName>robot_visual_3</visualName>
+        </visual>
+      </plugin>
     </model>
   </gazebo>
