Commit message: updated simulation with astra_cameras, frame changed to map instead of robot_map, changed the map file

File: rbares_description/robots/rbares_std.urdf.xacro (robot description, xacro)
@@ -8,4 +8,7 @@
   <!-- Import PALLET-TRUCK base elements -->
   <xacro:include filename="$(find rbares_description)/urdf/bases/rbares.urdf.xacro" />
+  <!-- Import orbbec embedded S camera and orbbec astra -->
+  <xacro:include filename="$(find rbares_description)/urdf/astra_camera/embedded_s.urdf.xacro" />
+  <xacro:include filename="$(find rbares_description)/urdf/astra_camera/orbbec_astra.urdf.xacro" />
   <!-- Import PALLET-TRUCK wheels -->
   <xacro:include filename="$(find rbares_description)/urdf/wheels/motor_wheel.urdf.xacro" />
@@ -109,13 +112,10 @@
       <origin xyz="${front_laser_x} ${front_laser_y} ${front_laser_z}" rpy="${PI} 0 0"/>
   </xacro:sensor_sick_s300>
-  <xacro:sensor_intel_d435 prefix="${prefix}left_fork_camera" parent="${prefix}left_fork_sensor_link" prefix_topic="${robot_id}/left_fork_camera" use_nominal_extrinsics="true" >
-        <origin xyz="0 0 0" rpy="0 -${5.0*PI/180.0} 0"/>
-  </xacro:sensor_intel_d435>
-  <xacro:sensor_intel_d435 prefix="${prefix}right_fork_camera" parent="${prefix}right_fork_sensor_link" prefix_topic="${robot_id}/right_fork_camera" use_nominal_extrinsics="true" >
-        <origin xyz="0 0 0" rpy="0 -${5.0*PI/180.0} 0"/>
-  </xacro:sensor_intel_d435>
-  <xacro:sensor_intel_d435 prefix="${prefix}rear_camera" parent="${prefix}rear_register_link" prefix_topic="${robot_id}/rear_camera" use_nominal_extrinsics="true" >
-        <origin xyz="0 0 0" rpy="0 ${5.0*PI/180.0} 0"/>
-  </xacro:sensor_intel_d435>
+  <xacro:orbbec_astra prefix="${prefix}rear_camera" parent="${prefix}rear_register_link" prefix_topic="${robot_id}/rear_camera">
+        <origin xyz="-0.019 0 0" rpy="0 0 0"/>
+  </xacro:orbbec_astra>
+  <xacro:sensor_orbbec_astra_embedded_s prefix="${prefix}left_fork_camera" parent="${prefix}left_fork_sensor_link" prefix_topic="${robot_id}/left_fork_camera" >
+        <origin xyz="0 0 0" rpy="0 0 0"/>
+  </xacro:sensor_orbbec_astra_embedded_s>
   <xacro:sensor_imu_hector prefix="${prefix}imu" parent="${prefix}base_link">
     <origin xyz="${imu_offset_x} -${imu_offset_y} ${imu_offset_z}" rpy="0 0 0"/>

File: rbares_description/urdf/bases/battery_case.urdf.xacro (robot description, xacro)
@@ -58,20 +58,4 @@
      <origin xyz="-0.439 0 -0.42" rpy="0 0 0" />
   </xacro:protection>
-  		<!--joint name="${prefix}right_projector_joint" type="fixed">
-  			<origin xyz="1 -1 1" rpy="0 0 0"/>
-  			<parent link="${prefix}battery_case_link"/>
-  			<child link="${prefix}right_line_projector"/>
-  		</joint>
-  		<link name="${prefix}right_line_projector">
-  		</link>
-  		<gazebo reference="${prefix}right_line_projector">
-  			<projector name="projector_test_right">
-  	    	<pose>0 0 0 1.57 0 0</pose>
-  	    	<texture>red1.png</texture>
-  	    	<fov>0.95</fov>
-  	    	<near_clip>0.1</near_clip>
-        	<far_clip>10.0</far_clip>
-  			</projector>
-  		</gazebo-->
   <!--gazebo reference="${prefix}battery_case_link">
     <mu1 value="1"/>

File: rbares_description/urdf/bases/front_case.urdf.xacro (robot description, xacro)
@@ -42,14 +42,12 @@
        </collision>
      </link>
-		 <xacro:line_projector prefix="${prefix}left_" parent="${prefix}front_case_link">
+		 <!--xacro:line_projector prefix="${prefix}left_" parent="${prefix}front_case_link">
 	      <origin xyz="0.2 -0.5 0.2" rpy="0 0 0" />
 	   </xacro:line_projector>
 		 <xacro:line_projector prefix="${prefix}right_" parent="${prefix}battery_case_link">
 				<origin xyz="0.1993 0.43 0.197" rpy="0 0 0" />
-		 </xacro:line_projector>
+		 </xacro:line_projector-->
 		 <!--xacro:led prefix="${prefix}">
 		 </xacro:led-->
-		 <xacro:led prefix="${prefix}">
-		 </xacro:led>
   </xacro:macro>
 </robot>

Commit message: rbares_description: updated to v2, added color and changed required positions

File: rbares_description/robots/rbares_std.urdf.xacro (robot description, xacro)
@@ -29,7 +29,7 @@
   <!-- Wheel parameters -->
   <!-- x,y,z in translation from base_link to the center of the wheel -->
-  <xacro:property name="wheel_offset_x" value="0.077"/>
+  <xacro:property name="wheel_offset_x" value="0.09139"/>
   <xacro:property name="wheel_offset_y" value="0.0"/>
-  <xacro:property name="wheel_offset_z" value="-0.59"/>
+  <xacro:property name="wheel_offset_z" value="-0.59825"/>
   <!-- Fork wheel -->
   <xacro:property name="fork_wheel_offset_x" value="0.0"/>
@@ -37,15 +37,15 @@
   <xacro:property name="fork_wheel_offset_z" value="0.0"/>
   <!-- Battery_case -->
-  <xacro:property name="battery_case_offset_x" value="1.2975"/>
+  <xacro:property name="battery_case_offset_x" value="1.2955"/>
   <xacro:property name="battery_case_offset_y" value="0.0"/>
-  <xacro:property name="battery_case_offset_z" value="0.674"/>
+  <xacro:property name="battery_case_offset_z" value="0.685"/>
   <!-- Front_case -->
-  <xacro:property name="front_case_offset_x" value="1.2982"/>
+  <xacro:property name="front_case_offset_x" value="1.2955"/>
   <xacro:property name="front_case_offset_y" value="0.0"/>
-  <xacro:property name="front_case_offset_z" value="0.671"/>
+  <xacro:property name="front_case_offset_z" value="0.685"/>
   <!-- Front support wheel -->
-  <xacro:property name="front_support_wheel_offset_x" value="0.340"/>
-  <xacro:property name="front_support_wheel_offset_y" value="0.180"/>
-  <xacro:property name="front_support_wheel_offset_z" value="-0.675"/>
+  <xacro:property name="front_support_wheel_offset_x" value="0.09139"/>
+  <xacro:property name="front_support_wheel_offset_y" value="0.224"/>
+  <xacro:property name="front_support_wheel_offset_z" value="-0.690"/>
   <!--  FORK CAMERAS  -->
   <xacro:property name="fork_camera_x" value="1.545" />
@@ -57,7 +57,7 @@
   <xacro:property name="front_laser_z" value="-0.38735" />
   <!-- RS_lIDAR -->
-  <xacro:property name="top_lidar_offset_x" value="0.085" />
+  <xacro:property name="top_lidar_offset_x" value="0.100" />
   <xacro:property name="top_lidar_offset_y" value="0.0" />
-  <xacro:property name="top_lidar_offset_z" value="0.205" />
+  <xacro:property name="top_lidar_offset_z" value="0.384" />
   <!-- REGISTERS -->
   <xacro:property name="front_register_offset_x" value="0.452" />

File: rbares_description/urdf/bases/battery_case.urdf.xacro (robot description, xacro)
@@ -4,12 +4,12 @@
   <xacro:include filename="$(find rbares_description)/urdf/elevator/fork.urdf.xacro" />
   <xacro:include filename="$(find rbares_description)/urdf/bases/protection.urdf.xacro" />
-      <!-- Robot mechanical and motor parameters -->
+  <!-- Robot mechanical and motor parameters -->
   <xacro:property name="battery_case_mass" value="10"/>
   <xacro:property name="battery_case_size_x" value="0.38"/>
   <xacro:property name="battery_case_size_y" value="0.57"/>
   <xacro:property name="battery_case_size_z" value="0.68"/>
-  <xacro:property name="fork_offset_x" value="-0.4325"/>
+  <xacro:property name="fork_offset_x" value="-0.4305"/>
   <xacro:property name="fork_offset_y" value="0.201"/>
-  <xacro:property name="fork_offset_z" value="-0.662"/>
+  <xacro:property name="fork_offset_z" value="-0.673"/>
   <xacro:property name="PI" value="3.1415926535897931"/>
   <xacro:macro name="solid_cuboid_inertia" params="m h d w">
@@ -31,5 +31,5 @@
       <origin xyz="0 0 0" rpy="0 0 0" />
       <geometry>
-        <mesh filename="package://rbares_description/meshes/bases/battery_case.stl"/>
+        <mesh filename="package://rbares_description/meshes/bases/battery_case_v2.stl"/>
       </geometry>
       <material name="dark_grey">
@@ -40,5 +40,5 @@
       <origin xyz="0 0 0" rpy="0 0 0" />
       <geometry>
-        <mesh filename="package://rbares_description/meshes/bases/battery_case.stl"/>
+           <mesh filename="package://rbares_description/meshes/bases/battery_case_v2.stl"/>
       </geometry>
     </collision>
@@ -58,11 +58,14 @@
      <origin xyz="-0.439 0 -0.42" rpy="0 0 0" />
   </xacro:protection>
-  <!--gazebo reference="${prefix}battery_case_link">
-    <mu1 value="1"/>
-    <mu2 value="1"/>
-    <!- -kp>100000000.0</kp- ->
-    <!- -kd value="10.0"/- ->
-    <material>Gazebo/Black</material>
-  </gazebo-->
+    <gazebo reference="${prefix}battery_case_link">
+      <visual>
+        <material>
+          <ambient>0.0 0.0 0.0 1.0</ambient>
+          <diffuse>0.2 0.2 0.2 1.0</diffuse>
+          <specular>0.508273 0.508273 0.508273 1.0</specular>
+          <emissive>0.0 0.0 0.0 0.0</emissive>
+        </material>
+      </visual>
+    </gazebo>
   <transmission name="${prefix}elevator_transmission">
     <type>transmission_interface/SimpleTransmission</type>

File: rbares_description/urdf/bases/front_case.urdf.xacro (robot description, xacro)
@@ -29,5 +29,5 @@
          <origin xyz="0 0 0" rpy="0 0 0" />
          <geometry>
-           <mesh filename="package://rbares_description/meshes/bases/front_case.stl"/>
+           <mesh filename="package://rbares_description/meshes/bases/front_case_v2.stl"/>
          </geometry>
          <material name="dark_grey">
@@ -38,5 +38,5 @@
          <origin xyz="0 0 0" rpy="0 0 0" />
          <geometry>
-           <mesh filename="package://rbares_description/meshes/bases/front_case.stl"/>
+           <mesh filename="package://rbares_description/meshes/bases/front_case_v2.stl"/>
          </geometry>
        </collision>
@@ -50,4 +50,14 @@
 		 <!--xacro:led prefix="${prefix}">
 		 </xacro:led-->
+    <gazebo reference="${prefix}front_case_link">
+      <visual>
+        <material>
+          <ambient>0.0 0.0 0.0 1.0</ambient>
+          <diffuse>0.2 0.2 0.2 1.0</diffuse>
+          <specular>0.508273 0.508273 0.508273 1.0</specular>
+          <emissive>0.0 0.0 0.0 0.0</emissive>
+        </material>
+      </visual>
+    </gazebo>
   </xacro:macro>
 </robot>

File: rbares_description/urdf/elevator/fork.urdf.xacro (robot description, xacro)
@@ -60,4 +60,12 @@
        <mu1>100</mu1>
        <mu2>100</mu2>
+       <visual>
+        <material>
+          <ambient>0.0 0.0 0.0 1.0</ambient>
+          <diffuse>0.2 0.2 0.2 1.0</diffuse>
+          <specular>0.508273 0.508273 0.508273 1.0</specular>
+          <emissive>0.0 0.0 0.0 0.0</emissive>
+        </material>
+      </visual>
      </gazebo>
     <joint name="${prefix}fork_sensor_joint" type="fixed">

File: rbares_description/urdf/wheels/castor_wheel.urdf.xacro (robot description, xacro)
@@ -3,5 +3,5 @@
   <xacro:property name="M_PI" value="3.1415926535897931" />
   <!-- Wheels -->
-  <xacro:property name="castor_wheel_radius" value="0.040" />
+  <xacro:property name="castor_wheel_radius" value="0.03" />
   <xacro:property name="castor_wheel_height" value="0.080" />
   <xacro:property name="castor_wheel_mass" value="0.5" />
@@ -26,5 +26,5 @@
         <origin xyz="0 0 0" rpy="0 0 0" />
         <geometry>
-		  <!--mesh filename="package://rbares_description/meshes/wheels/rbares_wheel_fake.dae"/-->
+		      <!--mesh filename="package://rbares_description/meshes/wheels/rbares_wheel_fake.dae"/-->
           <sphere radius="${castor_wheel_radius}"/>
         </geometry>
@@ -60,4 +60,12 @@
 		    <fdir1 value="1 0 0"/>
         <turnGravityOff>false</turnGravityOff>
+      <visual>
+        <material>
+          <ambient>0.0 0.0 0.0 1.0</ambient>
+          <diffuse>0.2 0.2 0.2 1.0</diffuse>
+          <specular>0.508273 0.508273 0.508273 1.0</specular>
+          <emissive>0.0 0.0 0.0 0.0</emissive>
+        </material>
+      </visual>
     </gazebo>
   </xacro:macro>

Commit message: rbares_description: removed intel cameras from robot file

File: rbares_description/robots/rbares_std.urdf.xacro (robot description, xacro)
@@ -109,13 +109,13 @@
       <origin xyz="${front_laser_x} ${front_laser_y} ${front_laser_z}" rpy="${PI} 0 0"/>
   </xacro:sensor_sick_s300>
-  <xacro:sensor_intel_d435 prefix="${prefix}left_fork_camera" parent="${prefix}left_fork_sensor_link" prefix_topic="${robot_id}/left_fork_camera" use_nominal_extrinsics="true" >
+  <!--xacro:sensor_intel_d435 prefix="${prefix}left_fork_camera" parent="${prefix}left_fork_sensor_link" prefix_topic="${robot_id}/left_fork_camera" use_nominal_extrinsics="true" >
         <origin xyz="0 0 0" rpy="0 -${5.0*PI/180.0} 0"/>
   </xacro:sensor_intel_d435>
   <xacro:sensor_intel_d435 prefix="${prefix}right_fork_camera" parent="${prefix}right_fork_sensor_link" prefix_topic="${robot_id}/right_fork_camera" use_nominal_extrinsics="true" >
         <origin xyz="0 0 0" rpy="0 -${5.0*PI/180.0} 0"/>
-  </xacro:sensor_intel_d435>
-  <xacro:sensor_intel_d435 prefix="${prefix}rear_camera" parent="${prefix}rear_register_link" prefix_topic="${robot_id}/rear_camera" use_nominal_extrinsics="true" >
-        <origin xyz="0 0 0" rpy="0 ${5.0*PI/180.0} 0"/>
-  </xacro:sensor_intel_d435>
+  </xacro:sensor_intel_d435-->
+  <!--xacro:sensor_intel_d435 prefix="${prefix}rear_camera" parent="${prefix}rear_register_link" prefix_topic="${robot_id}/rear_camera" use_nominal_extrinsics="true" >
+        <origin xyz="0.07 0 0" rpy="0 ${5.0*PI/180.0} 0"/>
+  </xacro:sensor_intel_d435-->
   <xacro:sensor_imu_hector prefix="${prefix}imu" parent="${prefix}base_link">
     <origin xyz="${imu_offset_x} -${imu_offset_y} ${imu_offset_z}" rpy="0 0 0"/>

Commit message: rbares_description:removed intel cameras

File: rbares_description/robots/rbares_std.urdf.xacro (robot description, xacro)
@@ -109,13 +109,7 @@
       <origin xyz="${front_laser_x} ${front_laser_y} ${front_laser_z}" rpy="${PI} 0 0"/>
   </xacro:sensor_sick_s300>
-  <xacro:sensor_intel_d435 prefix="${prefix}left_fork_camera" parent="${prefix}left_fork_sensor_link" prefix_topic="${robot_id}/left_fork_camera" use_nominal_extrinsics="true" >
-        <origin xyz="0 0 0" rpy="0 -${5.0*PI/180.0} 0"/>
-  </xacro:sensor_intel_d435>
-  <xacro:sensor_intel_d435 prefix="${prefix}right_fork_camera" parent="${prefix}right_fork_sensor_link" prefix_topic="${robot_id}/right_fork_camera" use_nominal_extrinsics="true" >
-        <origin xyz="0 0 0" rpy="0 -${5.0*PI/180.0} 0"/>
-  </xacro:sensor_intel_d435>
-  <xacro:sensor_intel_d435 prefix="${prefix}rear_camera" parent="${prefix}rear_register_link" prefix_topic="${robot_id}/rear_camera" use_nominal_extrinsics="true" >
-        <origin xyz="0 0 0" rpy="0 ${5.0*PI/180.0} 0"/>
-  </xacro:sensor_intel_d435>
+  <!--xacro:sensor_intel_d435 prefix="${prefix}rear_camera" parent="${prefix}rear_register_link" prefix_topic="${robot_id}/rear_camera" use_nominal_extrinsics="true" >
+        <origin xyz="0.07 0 0" rpy="0 ${5.0*PI/180.0} 0"/>
+  </xacro:sensor_intel_d435-->
   <xacro:sensor_imu_hector prefix="${prefix}imu" parent="${prefix}base_link">
     <origin xyz="${imu_offset_x} -${imu_offset_y} ${imu_offset_z}" rpy="0 0 0"/>

Commit message: rbares_description: updated locations and added color

File: rbares_description/robots/rbares_std.urdf.xacro (robot description, xacro)
@@ -26,7 +26,7 @@
   <!-- Wheel parameters -->
   <!-- x,y,z in translation from base_link to the center of the wheel -->
-  <xacro:property name="wheel_offset_x" value="0.077"/>
+  <xacro:property name="wheel_offset_x" value="0.09139"/>
   <xacro:property name="wheel_offset_y" value="0.0"/>
-  <xacro:property name="wheel_offset_z" value="-0.59"/>
+  <xacro:property name="wheel_offset_z" value="-0.59825"/>
   <!-- Fork wheel -->
   <xacro:property name="fork_wheel_offset_x" value="0.0"/>
@@ -34,15 +34,15 @@
   <xacro:property name="fork_wheel_offset_z" value="0.0"/>
   <!-- Battery_case -->
-  <xacro:property name="battery_case_offset_x" value="1.2975"/>
+  <xacro:property name="battery_case_offset_x" value="1.2955"/>
   <xacro:property name="battery_case_offset_y" value="0.0"/>
-  <xacro:property name="battery_case_offset_z" value="0.674"/>
+  <xacro:property name="battery_case_offset_z" value="0.685"/>
   <!-- Front_case -->
-  <xacro:property name="front_case_offset_x" value="1.2982"/>
+  <xacro:property name="front_case_offset_x" value="1.2955"/>
   <xacro:property name="front_case_offset_y" value="0.0"/>
-  <xacro:property name="front_case_offset_z" value="0.671"/>
+  <xacro:property name="front_case_offset_z" value="0.685"/>
   <!-- Front support wheel -->
-  <xacro:property name="front_support_wheel_offset_x" value="0.340"/>
-  <xacro:property name="front_support_wheel_offset_y" value="0.180"/>
-  <xacro:property name="front_support_wheel_offset_z" value="-0.675"/>
+  <xacro:property name="front_support_wheel_offset_x" value="0.09139"/>
+  <xacro:property name="front_support_wheel_offset_y" value="0.224"/>
+  <xacro:property name="front_support_wheel_offset_z" value="-0.690"/>
   <!--  FORK CAMERAS  -->
   <xacro:property name="fork_camera_x" value="1.545" />
@@ -54,7 +54,7 @@
   <xacro:property name="front_laser_z" value="-0.38735" />
   <!-- RS_lIDAR -->
-  <xacro:property name="top_lidar_offset_x" value="0.085" />
+  <xacro:property name="top_lidar_offset_x" value="0.100" />
   <xacro:property name="top_lidar_offset_y" value="0.0" />
-  <xacro:property name="top_lidar_offset_z" value="0.205" />
+  <xacro:property name="top_lidar_offset_z" value="0.384" />
   <!-- REGISTERS -->
   <xacro:property name="front_register_offset_x" value="0.452" />

File: rbares_description/urdf/bases/battery_case.urdf.xacro (robot description, xacro)
@@ -4,12 +4,12 @@
   <xacro:include filename="$(find rbares_description)/urdf/elevator/fork.urdf.xacro" />
   <xacro:include filename="$(find rbares_description)/urdf/bases/protection.urdf.xacro" />
-      <!-- Robot mechanical and motor parameters -->
+  <!-- Robot mechanical and motor parameters -->
   <xacro:property name="battery_case_mass" value="10"/>
   <xacro:property name="battery_case_size_x" value="0.38"/>
   <xacro:property name="battery_case_size_y" value="0.57"/>
   <xacro:property name="battery_case_size_z" value="0.68"/>
-  <xacro:property name="fork_offset_x" value="-0.4325"/>
+  <xacro:property name="fork_offset_x" value="-0.4305"/>
   <xacro:property name="fork_offset_y" value="0.201"/>
-  <xacro:property name="fork_offset_z" value="-0.662"/>
+  <xacro:property name="fork_offset_z" value="-0.673"/>
   <xacro:property name="PI" value="3.1415926535897931"/>
   <xacro:macro name="solid_cuboid_inertia" params="m h d w">
@@ -32,5 +32,5 @@
       <origin xyz="0 0 0" rpy="0 0 0" />
       <geometry>
-        <mesh filename="package://rbares_description/meshes/bases/battery_case.stl"/>
+        <mesh filename="package://rbares_description/meshes/bases/battery_case_v2.stl"/>
       </geometry>
       <material name="dark_grey">
@@ -41,5 +41,5 @@
       <origin xyz="0 0 0" rpy="0 0 0" />
       <geometry>
-        <mesh filename="package://rbares_description/meshes/bases/battery_case.stl"/>
+           <mesh filename="package://rbares_description/meshes/bases/battery_case_v2.stl"/>
       </geometry>
     </collision>
@@ -59,27 +59,14 @@
      <origin xyz="-0.439 0 -0.42" rpy="0 0 0" />
   </xacro:protection>
-  		<!--joint name="${prefix}right_projector_joint" type="fixed">
-  			<origin xyz="1 -1 1" rpy="0 0 0"/>
-  			<parent link="${prefix}battery_case_link"/>
-  			<child link="${prefix}right_line_projector"/>
-  		</joint>
-  		<link name="${prefix}right_line_projector">
-  		</link>
-  		<gazebo reference="${prefix}right_line_projector">
-  			<projector name="projector_test_right">
-  	    	<pose>0 0 0 1.57 0 0</pose>
-  	    	<texture>red1.png</texture>
-  	    	<fov>0.95</fov>
-  	    	<near_clip>0.1</near_clip>
-        	<far_clip>10.0</far_clip>
-  			</projector>
-  		</gazebo-->
-  <!--gazebo reference="${prefix}battery_case_link">
-    <mu1 value="1"/>
-    <mu2 value="1"/>
-    <!- -kp>100000000.0</kp- ->
-    <!- -kd value="10.0"/- ->
-    <material>Gazebo/Black</material>
-  </gazebo-->
+    <gazebo reference="${prefix}battery_case_link">
+      <visual>
+        <material>
+          <ambient>0.0 0.0 0.0 1.0</ambient>
+          <diffuse>0.2 0.2 0.2 1.0</diffuse>
+          <specular>0.508273 0.508273 0.508273 1.0</specular>
+          <emissive>0.0 0.0 0.0 0.0</emissive>
+        </material>
+      </visual>
+    </gazebo>
   <transmission name="${prefix}elevator_transmission">
     <type>transmission_interface/SimpleTransmission</type>

File: rbares_description/urdf/bases/front_case.urdf.xacro (robot description, xacro)
@@ -29,5 +29,5 @@
          <origin xyz="0 0 0" rpy="0 0 0" />
          <geometry>
-           <mesh filename="package://rbares_description/meshes/bases/front_case.stl"/>
+           <mesh filename="package://rbares_description/meshes/bases/front_case_v2.stl"/>
          </geometry>
          <material name="dark_grey">
@@ -38,18 +38,26 @@
          <origin xyz="0 0 0" rpy="0 0 0" />
          <geometry>
-           <mesh filename="package://rbares_description/meshes/bases/front_case.stl"/>
+           <mesh filename="package://rbares_description/meshes/bases/front_case_v2.stl"/>
          </geometry>
        </collision>
      </link>
-		 <xacro:line_projector prefix="${prefix}left_" parent="${prefix}front_case_link">
+		 <!--xacro:line_projector prefix="${prefix}left_" parent="${prefix}front_case_link">
 	      <origin xyz="0.2 -0.5 0.2" rpy="0 0 0" />
 	   </xacro:line_projector>
 		 <xacro:line_projector prefix="${prefix}right_" parent="${prefix}battery_case_link">
 				<origin xyz="0.1993 0.43 0.197" rpy="0 0 0" />
-		 </xacro:line_projector>
+		 </xacro:line_projector-->
 		 <!--xacro:led prefix="${prefix}">
 		 </xacro:led-->
-		 <xacro:led prefix="${prefix}">
-		 </xacro:led>
+    <gazebo reference="${prefix}front_case_link">
+      <visual>
+        <material>
+          <ambient>0.0 0.0 0.0 1.0</ambient>
+          <diffuse>0.2 0.2 0.2 1.0</diffuse>
+          <specular>0.508273 0.508273 0.508273 1.0</specular>
+          <emissive>0.0 0.0 0.0 0.0</emissive>
+        </material>
+      </visual>
+    </gazebo>
   </xacro:macro>
 </robot>

File: rbares_description/urdf/wheels/castor_wheel.urdf.xacro (robot description, xacro)
@@ -3,5 +3,5 @@
   <xacro:property name="M_PI" value="3.1415926535897931" />
   <!-- Wheels -->
-  <xacro:property name="castor_wheel_radius" value="0.040" />
+  <xacro:property name="castor_wheel_radius" value="0.03" />
   <xacro:property name="castor_wheel_height" value="0.080" />
   <xacro:property name="castor_wheel_mass" value="0.5" />
@@ -26,5 +26,5 @@
         <origin xyz="0 0 0" rpy="0 0 0" />
         <geometry>
-		  <!--mesh filename="package://rbares_description/meshes/wheels/rbares_wheel_fake.dae"/-->
+          <!--mesh filename="package://rbares_description/meshes/wheels/rbares_wheel_fake.dae"/-->
           <sphere radius="${castor_wheel_radius}"/>
         </geometry>
@@ -60,4 +60,12 @@
 		    <fdir1 value="1 0 0"/>
         <turnGravityOff>false</turnGravityOff>
+      <visual>
+        <material>
+          <ambient>0.0 0.0 0.0 1.0</ambient>
+          <diffuse>0.2 0.2 0.2 1.0</diffuse>
+          <specular>0.508273 0.508273 0.508273 1.0</specular>
+          <emissive>0.0 0.0 0.0 0.0</emissive>
+        </material>
+      </visual>
     </gazebo>
   </xacro:macro>
