Commit message: updated simulation and added new binaries

File: rbares_description/robots/rbares_std.urdf.xacro (robot description, xacro)
@@ -9,6 +9,6 @@
   <xacro:include filename="$(find rbares_description)/urdf/bases/rbares.urdf.xacro" />
   <!-- Import orbbec embedded S camera and orbbec astra -->
-  <!--xacro:include filename="$(find rbares_description)/urdf/astra_camera/embedded_s.urdf.xacro" />
-  <xacro:include filename="$(find rbares_description)/urdf/astra_camera/orbbec_astra.urdf.xacro" /-->
+  <xacro:include filename="$(find rbares_description)/urdf/astra_camera/embedded_s.urdf.xacro" />
+  <xacro:include filename="$(find rbares_description)/urdf/astra_camera/orbbec_astra.urdf.xacro" />
   <!-- Import PALLET-TRUCK wheels -->
   <xacro:include filename="$(find rbares_description)/urdf/wheels/motor_wheel.urdf.xacro" />
@@ -113,10 +113,10 @@
   </xacro:sensor_sick_s300>
   <!-- TODO: push orbbec on robotnik_sensor -->
-  <!--xacro:orbbec_astra prefix="${prefix}rear_camera" parent="${prefix}rear_register_link" prefix_topic="${robot_id}/rear_camera">
+  <xacro:orbbec_astra prefix="${prefix}rear_camera" parent="${prefix}rear_register_link" prefix_topic="${robot_id}/rear_camera">
         <origin xyz="-0.019 0 0" rpy="0 0 0"/>
   </xacro:orbbec_astra>
   <xacro:sensor_orbbec_astra_embedded_s prefix="${prefix}left_fork_camera" parent="${prefix}left_fork_sensor_link" prefix_topic="${robot_id}/left_fork_camera" >
         <origin xyz="0 0 0" rpy="0 0 0"/>
-  </xacro:sensor_orbbec_astra_embedded_s-->
+  </xacro:sensor_orbbec_astra_embedded_s>
   <xacro:sensor_imu_hector prefix="${prefix}imu" parent="${prefix}base_link">
     <origin xyz="${imu_offset_x} -${imu_offset_y} ${imu_offset_z}" rpy="0 0 0"/>

File: rbares_description/urdf/bases/rbares.urdf.xacro (robot description, xacro)
@@ -6,10 +6,5 @@
   <xacro:macro name="rbares" params="prefix publish_bf">
   <!-- BASE FOOTPRINT -->
-  <link name="${prefix}base_footprint">
-    <!--inertial>
-      <mass value="0.0001"/>
-      <inertia ixx="0.0001" ixy="0" ixz="0" iyy="0.0001" iyz="0" izz="0.0001"/>
-    </inertial-->
-  </link>
+  <link name="${prefix}base_footprint"/>
   <joint name="${prefix}base_footprint_joint" type="fixed">
     <origin xyz="${base_link_origin}" rpy="0 0 0" />

File: rbares_description/urdf/wheels/castor_wheel.urdf.xacro (robot description, xacro)
@@ -26,5 +26,5 @@
         <origin xyz="0 0 0" rpy="0 0 0" />
         <geometry>
-		      <!--mesh filename="package://rbares_description/meshes/wheels/rbares_wheel_fake.dae"/-->
+          <!--mesh filename="package://rbares_description/meshes/wheels/rbares_wheel_fake.dae"/-->
           <sphere radius="${castor_wheel_radius}"/>
         </geometry>

Commit message: changed parent link for the rear register

File: rbares_description/robots/rbares_std.urdf.xacro (robot description, xacro)
@@ -130,5 +130,5 @@
   <joint name="${prefix}rear_register_joint" type="fixed">
     <origin xyz="${rear_register_offset_x} ${rear_register_offset_y} ${rear_register_offset_z}" rpy="0 0 -${PI}"/>
-    <parent link="${prefix}front_case_link"/>
+    <parent link="${prefix}battery_case_link"/>
     <child link="${prefix}rear_register_link" />
   </joint>

Commit message: rbares_description: corrected typo

File: rbares_description/robots/rbares_std.urdf.xacro (robot description, xacro)
@@ -83,14 +83,14 @@
   <xacro:rbares prefix="${prefix}" publish_bf="true"/> <!-- BASE -->
   <xacro:motor_wheel prefix="${prefix}" parent="${prefix}front_case_link">
-      <origin xyz="${wheel_offset_x} ${wheel_offset_y} ${wheel_offset_z}" rpy="0 0 0"/>
+    <origin xyz="${wheel_offset_x} ${wheel_offset_y} ${wheel_offset_z}" rpy="0 0 0"/>
   </xacro:motor_wheel>
   <xacro:fork_wheel prefix="${prefix}left_fork_" parent="${prefix}base_link">
-      <origin xyz="${fork_wheel_offset_x} ${fork_wheel_offset_y} ${fork_wheel_offset_z}" rpy="0 0 0"/>
+    <origin xyz="${fork_wheel_offset_x} ${fork_wheel_offset_y} ${fork_wheel_offset_z}" rpy="0 0 0"/>
   </xacro:fork_wheel>
   <xacro:fork_wheel prefix="${prefix}right_fork_" parent="${prefix}base_link">
-      <origin xyz="${fork_wheel_offset_x} -${fork_wheel_offset_y} ${fork_wheel_offset_z}" rpy="0 0 0"/>
+    <origin xyz="${fork_wheel_offset_x} -${fork_wheel_offset_y} ${fork_wheel_offset_z}" rpy="0 0 0"/>
   </xacro:fork_wheel>
   <xacro:battery_case prefix="${prefix}" parent="${prefix}base_link">
-      <origin xyz="${battery_case_offset_x} -${battery_case_offset_y} ${battery_case_offset_z}" rpy="0 0 0"/>
+    <origin xyz="${battery_case_offset_x} -${battery_case_offset_y} ${battery_case_offset_z}" rpy="0 0 0"/>
   </xacro:battery_case>
   <xacro:front_case prefix="${prefix}" parent="${prefix}base_link">
@@ -98,20 +98,20 @@
   </xacro:front_case>
   <xacro:support_wheel prefix="${prefix}front_left_" parent="${prefix}front_case_link">
-      <origin xyz="${front_support_wheel_offset_x} ${front_support_wheel_offset_y} ${front_support_wheel_offset_z}" rpy="0 0 0"/>
+    <origin xyz="${front_support_wheel_offset_x} ${front_support_wheel_offset_y} ${front_support_wheel_offset_z}" rpy="0 0 0"/>
   </xacro:support_wheel>
   <xacro:support_wheel prefix="${prefix}front_right_" parent="${prefix}front_case_link">
-      <origin xyz="${front_support_wheel_offset_x} -${front_support_wheel_offset_y} ${front_support_wheel_offset_z}" rpy="0 0 0"/>
+    <origin xyz="${front_support_wheel_offset_x} -${front_support_wheel_offset_y} ${front_support_wheel_offset_z}" rpy="0 0 0"/>
   </xacro:support_wheel>
   <xacro:sensor_rslidar_16 prefix="${prefix}top_3d_lidar" parent="${prefix}front_case_link" prefix_topic="top_lidar" gpu="${gpu}">
-      <origin xyz="${top_lidar_offset_x} ${top_lidar_offset_y} ${top_lidar_offset_z}" rpy="0 0 0"/>
+    <origin xyz="${top_lidar_offset_x} ${top_lidar_offset_y} ${top_lidar_offset_z}" rpy="0 0 0"/>
   </xacro:sensor_rslidar_16>
   <xacro:sensor_sick_s300 prefix="${prefix}front_laser" parent="${prefix}front_case_link" prefix_topic="front_laser" min_angle="-2.35" max_angle="2.35" gpu="${gpu}" >
-      <origin xyz="${front_laser_x} ${front_laser_y} ${front_laser_z}" rpy="${PI} 0 0"/>
+    <origin xyz="${front_laser_x} ${front_laser_y} ${front_laser_z}" rpy="${PI} 0 0"/>
   </xacro:sensor_sick_s300>
   <xacro:sensor_orbbec_astra prefix="${prefix}rear_camera" parent="${prefix}rear_register_link" prefix_topic="${robot_id}/rear_camera">
-        <origin xyz="-0.019 0 0" rpy="0 0 0"/>
+    <origin xyz="-0.019 0 0" rpy="0 0 0"/>
   </xacro:sensor_orbbec_astra>
   <xacro:sensor_orbbec_astra_embedded_s prefix="${prefix}left_fork_camera" parent="${prefix}left_fork_sensor_link" prefix_topic="${robot_id}/left_fork_camera" >
-        <origin xyz="0 0 0" rpy="0 0 0"/>
+    <origin xyz="0 0 0" rpy="0 0 0"/>
   </xacro:sensor_orbbec_astra_embedded_s>
   <xacro:sensor_imu_hector prefix="${prefix}imu" parent="${prefix}base_link">

Commit message: rbares_description: remove xacro warnings in simulation

File: rbares_description/robots/rbares_std.urdf.xacro (robot description, xacro)
@@ -112,4 +112,7 @@
     <origin xyz="-0.019 0 0" rpy="0 0 0"/>
   </xacro:sensor_orbbec_astra>
+  <!--xacro:sensor_intel_d435 prefix="${prefix}mast_front_camera" parent="${prefix}base_link" prefix_topic="mast_front_camera">
+    <origin xyz="0 0 0" rpy="0 0 0"/>
+  </xacro:sensor_intel_d435-->
   <xacro:sensor_orbbec_astra_embedded_s prefix="${prefix}left_fork_camera" parent="${prefix}left_fork_sensor_link" prefix_topic="left_fork_camera" >
     <origin xyz="0 0 0" rpy="0 0 0"/>

File: rbares_description/urdf/bases/battery_case.urdf.xacro (robot description, xacro)
@@ -46,5 +46,5 @@
       <mass value="${battery_case_mass}" />
       <origin xyz="-0.2 0.0 -0.35"/>
-      <solid_cuboid_inertia m="${battery_case_mass}" h="${battery_case_size_y}" d="${battery_case_size_z}" w="${battery_case_size_x}"/>
+      <xacro:solid_cuboid_inertia m="${battery_case_mass}" h="${battery_case_size_y}" d="${battery_case_size_z}" w="${battery_case_size_x}"/>
     </inertial>
   </link>

File: rbares_description/urdf/bases/front_case.urdf.xacro (robot description, xacro)
@@ -24,5 +24,5 @@
          <mass value="${front_case_mass}" />
          <origin xyz="0.226093 0.0 -0.31"/>
-				 <solid_cuboid_inertia m="${front_case_mass}" h="${front_case_size_y}" d="${front_case_size_z}" w="${front_case_size_x}"/>
+	 <xacro:solid_cuboid_inertia m="${front_case_mass}" h="${front_case_size_y}" d="${front_case_size_z}" w="${front_case_size_x}"/>
        </inertial>
        <visual>

File: rbares_description/urdf/bases/mimic_base_link.urdf.xacro (robot description, xacro)
@@ -20,5 +20,5 @@
          <mass value="0.0001" />
          <origin xyz="0 0 0" rpy="0 0 0"/>
-				 <solid_cuboid_inertia m="0.0001" h="0.01" d="0.01" w="0.01"/>
+	 <xacro:solid_cuboid_inertia m="0.0001" h="0.01" d="0.01" w="0.01"/>
        </inertial>
      </link>

File: rbares_description/urdf/bases/protection.urdf.xacro (robot description, xacro)
@@ -17,5 +17,5 @@
        <mass value="0.01" />
        <origin xyz="0 0 0"/>
-       <solid_cuboid_inertia m="0.001" h="0.001" d="0.001" w="0.001"/>
+       <xacro:solid_cuboid_inertia m="0.001" h="0.001" d="0.001" w="0.001"/>
      </inertial>
    </link>

File: rbares_description/urdf/elevator/fork.urdf.xacro (robot description, xacro)
@@ -19,5 +19,5 @@
          <origin xyz="-0.381270 0.00000 0.012941" />
          <mass value="${fork_mass}" />
-         <solid_cuboid_inertia m="${fork_mass}" h="${fork_width}" d="${fork_height}" w="${fork_length}"/>
+         <xacro:solid_cuboid_inertia m="${fork_mass}" h="${fork_width}" d="${fork_height}" w="${fork_length}"/>
        </inertial>
        <visual>

File: rbares_description/urdf/epal_pallet/epal_pallet.urdf.xacro (robot description, xacro)
@@ -17,5 +17,5 @@
       <!-- yes, axis in solid_cuboid_inertia are changed, w relates to X axis, d to Z axis, and h to Y axis -->
       <!-- Keep this comment -->
-      <solid_cuboid_inertia m="5" h="0.044" d="0.8" w="1.2"/> <!-- h = z, d = y, w = x -->
+      <xacro:solid_cuboid_inertia m="5" h="0.044" d="0.8" w="1.2"/> <!-- h = z, d = y, w = x -->
     </inertial>
     <visual>
@@ -51,5 +51,5 @@
       <!-- yes, axis in solid_cuboid_inertia are changed, w relates to X axis, d to Z axis, and h to Y axis -->
       <!-- Keep this comment -->
-      <solid_cuboid_inertia m="1" h="0.1" d="0.1" w="1.2"/> <!-- h = z, d = y, w = x -->
+      <xacro:solid_cuboid_inertia m="1" h="0.1" d="0.1" w="1.2"/> <!-- h = z, d = y, w = x -->
     </inertial>
     <visual>
@@ -77,5 +77,5 @@
       <!-- yes, axis in solid_cuboid_inertia are changed, w relates to X axis, d to Z axis, and h to Y axis -->
       <!-- Keep this comment -->
-      <solid_cuboid_inertia m="1" h="0.1" d="0.1" w="1.2"/> <!-- h = z, d = y, w = x -->
+      <xacro:solid_cuboid_inertia m="1" h="0.1" d="0.1" w="1.2"/> <!-- h = z, d = y, w = x -->
     </inertial>
     <visual>
@@ -103,5 +103,5 @@
       <!-- yes, axis in solid_cuboid_inertia are changed, w relates to X axis, d to Z axis, and h to Y axis -->
       <!-- Keep this comment -->
-      <solid_cuboid_inertia m="1" h="0.1" d="0.1" w="1.2"/> <!-- h = z, d = y, w = x -->
+      <xacro:solid_cuboid_inertia m="1" h="0.1" d="0.1" w="1.2"/> <!-- h = z, d = y, w = x -->
     </inertial>
     <visual>

File: rbares_description/urdf/wheels/fork_wheel.urdf.xacro (robot description, xacro)
@@ -42,5 +42,5 @@
         <mass value="${fork_wheel_mass}" />
         <origin xyz="0 0 0" />
-        <cylinder_inertia  m="${fork_wheel_mass}" r="${fork_wheel_radius}" h="${fork_wheel_length}" />
+        <xacro:cylinder_inertia  m="${fork_wheel_mass}" r="${fork_wheel_radius}" h="${fork_wheel_length}" />
       </inertial>
     </link>

File: rbares_description/urdf/wheels/motor_wheel.urdf.xacro (robot description, xacro)
@@ -44,5 +44,5 @@
         <mass value="${wheel_mass}" />
         <origin xyz="0 0 0"/>
-        <cylinder_inertia m="${wheel_mass}" r="${wheel_width}" h="${wheel_radius}" />
+        <xacro:cylinder_inertia m="${wheel_mass}" r="${wheel_width}" h="${wheel_radius}" />
       </inertial>
     </link>
@@ -79,5 +79,5 @@
         <mass value="${wheel_mass}" />
         <origin xyz="0.000063 0 0.000465"/>
-        <cylinder_inertia  m="${wheel_mass}" r="${wheel_radius}" h="${wheel_width}" />
+        <xacro:cylinder_inertia  m="${wheel_mass}" r="${wheel_radius}" h="${wheel_width}" />
       </inertial>
     </link>
